File: rocket2-afs2-cleaned.kicad_sch (KiCad schematic)
At the start: 45 parts, among them J1 ARM Cortex Debug, U1 STM32F105RCT6, U2 LD1086DT33TR, U4 USBLC6-2SC6, U5 ADXL383, Y1 8MHz

Commit message: Tmp staging ground cleaned up with astra and then improved schematic some more
Parts:
- added J3: POWER, TerminalBlock:TerminalBlock_bornier-2_P5.08mm, symbol Connector:Conn_01x02_Socket
- added R7: 10K, Resistor_SMD:R_0402_1005Metric, symbol Device:R_Small_US
- J1: symbol UCIRP:ARM_Cortex_Debug -> UCIRP-KiCAD-Lib:ARM_Cortex_Debug
- U1: symbol UCIRP:MCU STM32F105RCT6 -> UCIRP-KiCAD-Lib:MCU STM32F105RCT6
- U3: symbol UCIRP:Flash_Memory W25N01GVZE -> UCIRP-KiCAD-Lib:Flash_Memory W25N01GVZE
- U30: symbol UCIRP-KiCAD-Lib:MAX31855 -> UCIRP-KiCAD-Lib:TC_ADC MAX31855JASA+
- U5: symbol UCIRP:ADXL383 -> UCIRP-KiCAD-Lib:ADXL383
- U6: symbol UCIRP-KiCAD-Lib:BMI088 -> UCIRP-KiCAD-Lib:IMU BMI088
- U7: symbol UCIRP-KiCAD-Lib:MS5607-02BA -> UCIRP-KiCAD-Lib:Altimeter MS5607-02BA
- Y1: Part # ECS-1633-160-BN-TR -> ASDMB-8-000MHZ-XY-T
- renumbered C2 to C14
Connections:
- net +3.3V: now also R7.1
- net GND: now also U2.1 (ADJ/GND), J3.2 (Pin_2)
- net IMU_INT1: now also U1.24 (PC4)
- net IMU_INT2: now also U1.25 (PC5)
- net IMU_INT3: now also U1.26 (PB0)
- net IMU_INT4: now also U1.29 (PB10)
- net MEM_~{HOLD}: now also R7.2
- net VCC: now also J3.1 (Pin_1)
- no-connect marks 17 -> 39
Other:
- note added: "01 MCU | STM32F105"
- note added: "02 3.3 V REGULATOR"
- note added: "03 CLOCK | 8 MHz"
- note added: "04 SPI FLASH"
- note added: "05 SWD DEBUG"
- note added: "06 BAROMETER | MS5607"
- note added: "07 THERMOCOUPLE | MAX31855"
- note added: "08 HIGH-G ACCELEROMETER | ADXL383"
- note added: "09 USB-C | DATA + VBUS SENSE"
- note added: "10 IMU | BMI088"
- note added: "11 PWR"
- note added: "CS pull-ups are grouped with their SPI devices."
- note added: "IMU Interrupts are placed weirdly so they each occupy their own EXTI bus"
- note added: "INT0: data ready INT1: threshold interrupt (firmware-defined)"
- note added: "MCU supply bypass capacitors"
- note removed: "Int0: Data ready Int1: Accel threshold reached or smth (arm/start)"
- title: (none) -> AFS2 | Flight Computer
- moved on the sheet: C1, C10, C11, C118, C12, C13, C14, C16, C18, C2, C21, C3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
