File: rocket2-afs2.kicad_pcb (KiCad board)
At the start: 2 copper layers, 54 x 54 mm, 52 parts, among them J1 ARM Cortex Debug, J3 XT60 POWER, U1 STM32F105RCT6, U2 LD1086DT33TR, U4 USBLC6-2SC6, U5 ADXL383, Y1 8MHz

Commit message: Ready for PDR. Might still mess around more but its all routed and passes
Parts:
- H1, H2, H3, H4: value M3 mounting hole -> MountingHole_Pad; footprint MountingHole:MountingHole_3.2mm_M3 -> MountingHole:MountingHole_3.2mm_M3_Pad_Via
- moved C12 1.53 mm to (108.7, 147.2), turned to 0 degrees
- moved C5 0.94 mm to (117.1, 131.1)
Routing:
- net +3.3V: track 46.8 -> 271.7 mm, vias 0 -> 9
- net GND: track 2.00 -> 0.00 mm, vias 124 -> 88
- net /IMU_INT3: track 14.9 -> 16.4 mm
- net /IMU_INT1: track 14.9 -> 15.5 mm
