File: rocket2-afs2.kicad_sch (KiCad schematic)
At the start: 45 parts, among them J1 ARM Cortex Debug, U1 STM32F105RCT6, U2 LD1086DT33TR, U4 USBLC6-2SC6, U5 ADXL383, Y1 8MHz

Commit message: Finished routing iteration 1. Going to try moving everything to the front next
Parts:
- added J3: XT60 POWER, Connector_AMASS:AMASS_XT60PW-M_1x02_P7.20mm_Horizontal, symbol Connector:Conn_01x02_Socket
- added R7: 10K, Resistor_SMD:R_0402_1005Metric, symbol Device:R_Small_US
- C1: Part # Generic 0603 6.3V 10uF X7R MLCC -> Generic 0603 16V 10uF X7R MLCC
- J1: symbol UCIRP:ARM_Cortex_Debug -> UCIRP-KiCAD-Lib:ARM_Cortex_Debug
- TC1: footprint 0UCIRP-KiCAD-Lib:AM-K-PCB -> 0UCIRP-KiCAD-Lib:TC_Connector AM-K-PCB
- U1: symbol UCIRP:MCU STM32F105RCT6 -> UCIRP-KiCAD-Lib:MCU STM32F105RCT6
- U3: symbol UCIRP:Flash_Memory W25N01GVZE -> UCIRP-KiCAD-Lib:Flash_Memory W25N01GVZE
- U30: symbol UCIRP-KiCAD-Lib:MAX31855 -> UCIRP-KiCAD-Lib:TC_ADC MAX31855JASA+
- U5: symbol UCIRP:ADXL383 -> UCIRP-KiCAD-Lib:ADXL383
- U6: footprint UCIRP-KiCAD-Lib:BMI088 -> 0UCIRP-KiCAD-Lib:IMU BMI088; symbol UCIRP-KiCAD-Lib:BMI088 -> UCIRP-KiCAD-Lib:IMU BMI088
- U7: footprint UCIRP-KiCAD-Lib:MS5607-02BA -> 0UCIRP-KiCAD-Lib:Altimeter MS5607-02BA; symbol UCIRP-KiCAD-Lib:MS5607-02BA -> UCIRP-KiCAD-Lib:Altimeter MS5607-02BA
- Y1: Part # ECS-1633-160-BN-TR -> ASDMB-8-000MHZ-XY-T
- renumbered C2 to C14
Connections:
- net +3.3V: now also R7.1
- net GND: now also U2.1 (ADJ/GND), J3.1 (Pin_1)
- net IMU_INT1: now also U1.24 (PC4)
- net IMU_INT3: now also U1.25 (PC5)
- net MEM_~{HOLD}: now also R7.2
- net VCC: now also J3.2 (Pin_2)
- no-connect marks 17 -> 33
Other:
- note added: "01 MCU | STM32F105"
- note added: "02 3.3 V REGULATOR"
- note added: "03 CLOCK | 8 MHz"
- note added: "04 SPI FLASH"
- note added: "05 SWD DEBUG"
- note added: "06 BAROMETER | MS5607"
- note added: "07 THERMOCOUPLE | MAX31855"
- note added: "08 HIGH-G ACCELEROMETER | ADXL383"
- note added: "09 USB-C | DATA + VBUS SENSE"
- note added: "10 IMU | BMI088"
- note added: "11 PWR"
- note added: "CS pull-ups are grouped with their SPI devices."
- note added: "IMU Interrupts are placed weirdly so they each occupy their own EXTI bus"
- note added: "INT0: data ready INT1: threshold interrupt (firmware-defined)"
- note added: "MCU supply bypass capacitors"
- note removed: "Int0: Data ready Int1: Accel threshold reached or smth (arm/start)"
- title: (none) -> AFS2 | Flight Computer
- moved on the sheet: C1, C10, C11, C118, C12, C13, C14, C16, C18, C2, C21, C3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

Commit message: Moved all to front
Connections:
- net ACCEL_INT0: now also U1.16 (PA2); no longer U1.15 (PA1)
- net ACCEL_INT1: now also U1.15 (PA1); no longer U1.16 (PA2)
Changed lines of the file:
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@@
-		)
-	)
-	(label "ACCEL_INT0"
-		(at 41.91 71.12 180)
-		(effects
-			(font
-				(size 1.27 1.27)
-			)
-			(justify right)
 		)
 	)
@@
 		)
 	)
+	(label "ACCEL_INT1"
+		(at 41.91 71.12 180)
+		(effects
+			(font
+				(size 1.27 1.27)
+			)
+			(justify right)
+		)
+	)
 	(label "TC_~{CS}"
 		(at 87.63 91.44 0)
@@
 		)
 	)
-	(label "ACCEL_INT1"
-		(at 41.91 73.66 180)
-		(effects
-			(font
-				(size 1.27 1.27)
-			)
-			(justify right)
-		)
-	)
 	(label "MEM_~{CS}"
 		(at 87.63 99.06 0)
@@
 		)
 	)
+	(label "ACCEL_INT0"
+		(at 41.91 73.66 180)
+		(effects
+			(font
+				(size 1.27 1.27)
+			)
+			(justify right)
+		)
+	)

Commit message: Ready for PDR. Might still mess around more but its all routed and passes
Parts:
- added H1, H2, H3, H4: MountingHole_Pad, MountingHole:MountingHole_3.2mm_M3_Pad_Via, symbol Mechanical:MountingHole_Pad
